Commit message: Updated models

File: iCub/robots/iCubDarmstadt01/model.urdf (robot description, URDF)
Before this commit: robot ICUB_2-5_BB_SIM_MODEL, 163 links, 162 joints
Links:
- removed link chest_ems_acc_eb1
- removed link chest_ems_acc_eb2
- removed link chest_ems_acc_eb3
- removed link chest_ems_acc_eb4
- removed link chest_ems_gyro_eb1
- removed link chest_ems_gyro_eb2
- removed link chest_ems_gyro_eb3
- removed link chest_ems_gyro_eb4
- removed link chest_mtb_acc_0b10
- removed link chest_mtb_acc_0b7
- removed link chest_mtb_acc_0b8
- removed link chest_mtb_acc_0b9
- removed link imu
- removed link l_foot_mtb_acc_10b12
- removed link l_foot_mtb_acc_10b13
- removed link l_forearm_mtb_acc_1b7
- removed link l_forearm_mtb_acc_1b8
- removed link l_forearm_mtb_acc_1b9
- removed link l_lower_leg_ems_acc_eb7
- removed link l_lower_leg_ems_gyro_eb7
- removed link l_lower_leg_mtb_acc_10b10
- removed link l_lower_leg_mtb_acc_10b11
- removed link l_lower_leg_mtb_acc_10b8
- removed link l_lower_leg_mtb_acc_10b9
- removed link l_upper_arm_mtb_acc_1b10
- removed link l_upper_arm_mtb_acc_1b11
- removed link l_upper_arm_mtb_acc_1b12
- removed link l_upper_arm_mtb_acc_1b13
- removed link l_upper_leg_ems_acc_eb10
- removed link l_upper_leg_ems_acc_eb6
- removed link l_upper_leg_ems_gyro_eb10
- removed link l_upper_leg_ems_gyro_eb6
- removed link l_upper_leg_mtb_acc_10b1
- removed link l_upper_leg_mtb_acc_10b2
- removed link l_upper_leg_mtb_acc_10b3
- removed link l_upper_leg_mtb_acc_10b4
- removed link l_upper_leg_mtb_acc_10b5
- removed link l_upper_leg_mtb_acc_10b6
- removed link l_upper_leg_mtb_acc_10b7
- removed link r_foot_mtb_acc_11b12
- removed link r_foot_mtb_acc_11b13
- removed link r_forearm_mtb_acc_2b7
- removed link r_forearm_mtb_acc_2b8
- removed link r_forearm_mtb_acc_2b9
- removed link r_lower_leg_ems_acc_eb9
- removed link r_lower_leg_ems_gyro_eb9
- removed link r_lower_leg_mtb_acc_11b10
- removed link r_lower_leg_mtb_acc_11b11
- removed link r_lower_leg_mtb_acc_11b8
- removed link r_lower_leg_mtb_acc_11b9
- removed link r_upper_arm_mtb_acc_2b10
- removed link r_upper_arm_mtb_acc_2b11
- removed link r_upper_arm_mtb_acc_2b12
- removed link r_upper_arm_mtb_acc_2b13
- removed link r_upper_leg_ems_acc_eb11
- removed link r_upper_leg_ems_acc_eb8
- removed link r_upper_leg_ems_gyro_eb11
- removed link r_upper_leg_ems_gyro_eb8
- removed link r_upper_leg_mtb_acc_11b1
- removed link r_upper_leg_mtb_acc_11b2
- removed link r_upper_leg_mtb_acc_11b3
- removed link r_upper_leg_mtb_acc_11b4
- removed link r_upper_leg_mtb_acc_11b5
- removed link r_upper_leg_mtb_acc_11b6
- removed link r_upper_leg_mtb_acc_11b7
- removed link root_link_ems_acc_eb5
- removed link root_link_ems_gyro_eb5
- added link imu_frame
- link chest: geometry collision mesh filename=package://iCub/meshes/simmechanics/sim_sea_2-5_chest_bb_prt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 scale=0.001 0.001 0.001; visual mesh filename=package://iCub/meshes/simmechanics/sim_sea_2-5_chest_bb_prt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 scale=0.001 0.001 0.001
- link head: geometry collision mesh filename=package://iCub/meshes/simmechanics/sim_sea_2-5_head_prt-bin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 scale=0.001 0.001 0.001; visual mesh filename=package://iCub/meshes/simmechanics/sim_sea_2-5_head_prt-bin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 scale=0.001 0.001 0.001
- link l_ankle_1: geometry collision mesh filename=package://iCub/meshes/simmechanics/sim_sea_2-5_l_ankle_prt-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 scale=0.001 0.001 0.001; visual mesh filename=package://iCub/meshes/simmechanics/sim_sea_2-5_l_ankle_prt-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 scale=0.001 0.001 0.001
- link l_ankle_2: geometry collision mesh filename=package://iCub/meshes/simmechanics/sim_sea_2-5_l_foot_prt-b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 scale=0.001 0.001 0.001; visual mesh filename=package://iCub/meshes/simmechanics/sim_sea_2-5_l_foot_prt-b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 scale=0.001 0.001 0.001
- link l_elbow_1: geometry collision mesh filename=package://iCub/meshes/simmechanics/sim_sea_2-5_l_elbow_pros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 scale=0.001 0.001 0.001; visual mesh filename=package://iCub/meshes/simmechanics/sim_sea_2-5_l_elbow_pros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 scale=0.001 0.001 0.001
- link l_foot: geometry collision mesh filename=package://iCub/meshes/simmechanics/sim_sea_2-5_l_sole_prt-b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 scale=0.001 0.001 0.001; visual mesh filename=package://iCub/meshes/simmechanics/sim_sea_2-5_l_sole_prt-b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 scale=0.001 0.001 0.001
- link l_forearm: geometry collision mesh filename=package://iCub/meshes/simmechanics/sim_sea_2-5_l_forearm_pr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 scale=0.001 0.001 0.001; visual mesh filename=package://iCub/meshes/simmechanics/sim_sea_2-5_l_forearm_pr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 scale=0.001 0.001 0.001
- link l_hand: geometry collision mesh filename=package://iCub/meshes/simmechanics/sim_sea_2-5_l_hand_prt-b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 scale=0.001 0.001 0.001; visual mesh filename=package://iCub/meshes/simmechanics/sim_sea_2-5_l_hand_prt-b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 scale=0.001 0.001 0.001
- link l_hip_1: geometry collision mesh filename=package://iCub/meshes/simmechanics/sim_sea_2-5_l_hip_1_prt-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 scale=0.001 0.001 0.001; visual mesh filename=package://iCub/meshes/simmechanics/sim_sea_2-5_l_hip_1_prt-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 scale=0.001 0.001 0.001
- link l_hip_2: geometry collision mesh filename=package://iCub/meshes/simmechanics/sim_sea_2-5_l_hip_2_prt-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 scale=0.001 0.001 0.001; visual mesh filename=package://iCub/meshes/simmechanics/sim_sea_2-5_l_hip_2_prt-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 scale=0.001 0.001 0.001
- link l_hip_3: geometry collision mesh filename=package://iCub/meshes/simmechanics/sim_sea_2-5_l_upper_thig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 scale=0.001 0.001 0.001; visual mesh filename=package://iCub/meshes/simmechanics/sim_sea_2-5_l_upper_thig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 scale=0.001 0.001 0.001
- link l_lower_leg: geometry collision mesh filename=package://iCub/meshes/simmechanics/sim_sea_2-5_l_shank_prt-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 scale=0.001 0.001 0.001; visual mesh filename=package://iCub/meshes/simmechanics/sim_sea_2-5_l_shank_prt-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 scale=0.001 0.001 0.001
- link l_shoulder_1: geometry collision mesh filename=package://iCub/meshes/simmechanics/sim_sea_2-5_l_shoulder_1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 scale=0.001 0.001 0.001; visual mesh filename=package://iCub/meshes/simmechanics/sim_sea_2-5_l_shoulder_1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 scale=0.001 0.001 0.001
- link l_shoulder_2: geometry collision mesh filename=package://iCub/meshes/simmechanics/sim_sea_2-5_l_shoulder_2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 scale=0.001 0.001 0.001; visual mesh filename=package://iCub/meshes/simmechanics/sim_sea_2-5_l_shoulder_2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 scale=0.001 0.001 0.001
- link l_shoulder_3: geometry collision mesh filename=package://iCub/meshes/simmechanics/sim_sea_2-5_l_upper_arm_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 scale=0.001 0.001 0.001; visual mesh filename=package://iCub/meshes/simmechanics/sim_sea_2-5_l_upper_arm_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 scale=0.001 0.001 0.001
- link l_upper_arm: geometry collision mesh filename=package://iCub/meshes/simmechanics/sim_sea_2-5_l_elbow_prt-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 scale=0.001 0.001 0.001; visual mesh filename=package://iCub/meshes/simmechanics/sim_sea_2-5_l_elbow_prt-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 scale=0.001 0.001 0.001
- link l_upper_leg: geometry collision mesh filename=package://iCub/meshes/simmechanics/sim_sea_2-5_l_thigh_prt-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 scale=0.001 0.001 0.001; visual mesh filename=package://iCub/meshes/simmechanics/sim_sea_2-5_l_thigh_prt-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 scale=0.001 0.001 0.001
- link l_wrist_1: geometry collision mesh filename=package://iCub/meshes/simmechanics/sim_sea_2-5_l_wrist_pitc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 scale=0.001 0.001 0.001; visual mesh filename=package://iCub/meshes/simmechanics/sim_sea_2-5_l_wrist_pitc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 scale=0.001 0.001 0.001
- link neck_1: geometry collision mesh filename=package://iCub/meshes/simmechanics/sim_sea_2-5_neck_1_prt-b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 scale=0.001 0.001 0.001; visual mesh filename=package://iCub/meshes/simmechanics/sim_sea_2-5_neck_1_prt-b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 scale=0.001 0.001 0.001
- link neck_2: geometry collision mesh filename=package://iCub/meshes/simmechanics/sim_sea_2-5_neck_2_prt-b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 scale=0.001 0.001 0.001; visual mesh filename=package://iCub/meshes/simmechanics/sim_sea_2-5_neck_2_prt-b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 scale=0.001 0.001 0.001
- link r_ankle_1: geometry collision mesh filename=package://iCub/meshes/simmechanics/sim_sea_2-5_r_ankle_prt-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 scale=0.001 0.001 0.001; visual mesh filename=package://iCub/meshes/simmechanics/sim_sea_2-5_r_ankle_prt-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 scale=0.001 0.001 0.001
- link r_ankle_2: geometry collision mesh filename=package://iCub/meshes/simmechanics/sim_sea_2-5_r_foot_prt-b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 scale=0.001 0.001 0.001; visual mesh filename=package://iCub/meshes/simmechanics/sim_sea_2-5_r_foot_prt-b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 scale=0.001 0.001 0.001
- link r_elbow_1: geometry collision mesh filename=package://iCub/meshes/simmechanics/sim_sea_2-5_r_elbow_pros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 scale=0.001 0.001 0.001; visual mesh filename=package://iCub/meshes/simmechanics/sim_sea_2-5_r_elbow_pros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 scale=0.001 0.001 0.001
- link r_foot: geometry collision mesh filename=package://iCub/meshes/simmechanics/sim_sea_2-5_r_sole_prt-b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 scale=0.001 0.001 0.001; visual mesh filename=package://iCub/meshes/simmechanics/sim_sea_2-5_r_sole_prt-b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 scale=0.001 0.001 0.001
- link r_forearm: geometry collision mesh filename=package://iCub/meshes/simmechanics/sim_sea_2-5_r_forearm_pr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 scale=0.001 0.001 0.001; visual mesh filename=package://iCub/meshes/simmechanics/sim_sea_2-5_r_forearm_pr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 scale=0.001 0.001 0.001
- link r_hand: geometry collision mesh filename=package://iCub/meshes/simmechanics/sim_sea_2-5_r_hand_prt-b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 scale=0.001 0.001 0.001; visual mesh filename=package://iCub/meshes/simmechanics/sim_sea_2-5_r_hand_prt-b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 scale=0.001 0.001 0.001
- link r_hip_1: geometry collision mesh filename=package://iCub/meshes/simmechanics/sim_sea_2-5_r_hip_1_prt-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 scale=0.001 0.001 0.001; visual mesh filename=package://iCub/meshes/simmechanics/sim_sea_2-5_r_hip_1_prt-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 scale=0.001 0.001 0.001
- link r_hip_2: geometry collision mesh filename=package://iCub/meshes/simmechanics/sim_sea_2-5_r_hip_2_prt-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 scale=0.001 0.001 0.001; visual mesh filename=package://iCub/meshes/simmechanics/sim_sea_2-5_r_hip_2_prt-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 scale=0.001 0.001 0.001
- link r_hip_3: geometry collision mesh filename=package://iCub/meshes/simmechanics/sim_sea_2-5_r_upper_thig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 scale=0.001 0.001 0.001; visual mesh filename=package://iCub/meshes/simmechanics/sim_sea_2-5_r_upper_thig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 scale=0.001 0.001 0.001
- link r_lower_leg: geometry collision mesh filename=package://iCub/meshes/simmechanics/sim_sea_2-5_r_shank_prt-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 scale=0.001 0.001 0.001; visual mesh filename=package://iCub/meshes/simmechanics/sim_sea_2-5_r_shank_prt-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 scale=0.001 0.001 0.001
- link r_shoulder_1: geometry collision mesh filename=package://iCub/meshes/simmechanics/sim_sea_2-5_r_shoulder_1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 scale=0.001 0.001 0.001; visual mesh filename=package://iCub/meshes/simmechanics/sim_sea_2-5_r_shoulder_1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 scale=0.001 0.001 0.001
- link r_shoulder_2: geometry collision mesh filename=package://iCub/meshes/simmechanics/sim_sea_2-5_r_shoulder_2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 scale=0.001 0.001 0.001; visual mesh filename=package://iCub/meshes/simmechanics/sim_sea_2-5_r_shoulder_2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 scale=0.001 0.001 0.001
- link r_shoulder_3: geometry collision mesh filename=package://iCub/meshes/simmechanics/sim_sea_2-5_r_upper_arm_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 scale=0.001 0.001 0.001; visual mesh filename=package://iCub/meshes/simmechanics/sim_sea_2-5_r_upper_arm_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 scale=0.001 0.001 0.001
- link r_upper_arm: geometry collision mesh filename=package://iCub/meshes/simmechanics/sim_sea_2-5_r_elbow_prt-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 scale=0.001 0.001 0.001; visual mesh filename=package://iCub/meshes/simmechanics/sim_sea_2-5_r_elbow_prt-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 scale=0.001 0.001 0.001
- link r_upper_leg: geometry collision mesh filename=package://iCub/meshes/simmechanics/sim_sea_2-5_r_thigh_prt-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 scale=0.001 0.001 0.001; visual mesh filename=package://iCub/meshes/simmechanics/sim_sea_2-5_r_thigh_prt-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 scale=0.001 0.001 0.001
- link r_wrist_1: geometry collision mesh filename=package://iCub/meshes/simmechanics/sim_sea_2-5_r_wrist_pitc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 scale=0.001 0.001 0.001; visual mesh filename=package://iCub/meshes/simmechanics/sim_sea_2-5_r_wrist_pitc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 scale=0.001 0.001 0.001
- link root_link: geometry collision mesh filename=package://iCub/meshes/simmechanics/sim_sea_2-5_root_link_pr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 scale=0.001 0.001 0.001; visual mesh filename=package://iCub/meshes/simmechanics/sim_sea_2-5_root_link_pr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 scale=0.001 0.001 0.001
- link torso_1: geometry collision mesh filename=package://iCub/meshes/simmechanics/sim_sea_2-5_lap_belt_1_p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 scale=0.001 0.001 0.001; visual mesh filename=package://iCub/meshes/simmechanics/sim_sea_2-5_lap_belt_1_p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 scale=0.001 0.001 0.001
- link torso_2: geometry collision mesh filename=package://iCub/meshes/simmechanics/sim_sea_2-5_lap_belt_2_p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 scale=0.001 0.001 0.001; visual mesh filename=package://iCub/meshes/simmechanics/sim_sea_2-5_lap_belt_2_p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 scale=0.001 0.001 0.001
Joints:
- removed joint chest_ems_acc_eb1_fixed_joint
- removed joint chest_ems_acc_eb2_fixed_joint
- removed joint chest_ems_acc_eb3_fixed_joint
- removed joint chest_ems_acc_eb4_fixed_joint
- removed joint chest_ems_gyro_eb1_fixed_joint
- removed joint chest_ems_gyro_eb2_fixed_joint
- removed joint chest_ems_gyro_eb3_fixed_joint
- removed joint chest_ems_gyro_eb4_fixed_joint
- removed joint chest_mtb_acc_0b10_fixed_joint
- removed joint chest_mtb_acc_0b7_fixed_joint
- removed joint chest_mtb_acc_0b8_fixed_joint
- removed joint chest_mtb_acc_0b9_fixed_joint
- removed joint imu_fixed_joint
- removed joint l_foot_mtb_acc_10b12_fixed_joint
- removed joint l_foot_mtb_acc_10b13_fixed_joint
- removed joint l_forearm_mtb_acc_1b7_fixed_joint
- removed joint l_forearm_mtb_acc_1b8_fixed_joint
- removed joint l_forearm_mtb_acc_1b9_fixed_joint
- removed joint l_lower_leg_ems_acc_eb7_fixed_joint
- removed joint l_lower_leg_ems_gyro_eb7_fixed_joint
- removed joint l_lower_leg_mtb_acc_10b10_fixed_joint
- removed joint l_lower_leg_mtb_acc_10b11_fixed_joint
- removed joint l_lower_leg_mtb_acc_10b8_fixed_joint
- removed joint l_lower_leg_mtb_acc_10b9_fixed_joint
- removed joint l_upper_arm_mtb_acc_1b10_fixed_joint
- removed joint l_upper_arm_mtb_acc_1b11_fixed_joint
- removed joint l_upper_arm_mtb_acc_1b12_fixed_joint
- removed joint l_upper_arm_mtb_acc_1b13_fixed_joint
- removed joint l_upper_leg_ems_acc_eb10_fixed_joint
- removed joint l_upper_leg_ems_acc_eb6_fixed_joint
- removed joint l_upper_leg_ems_gyro_eb10_fixed_joint
- removed joint l_upper_leg_ems_gyro_eb6_fixed_joint
- removed joint l_upper_leg_mtb_acc_10b1_fixed_joint
- removed joint l_upper_leg_mtb_acc_10b2_fixed_joint
- removed joint l_upper_leg_mtb_acc_10b3_fixed_joint
- removed joint l_upper_leg_mtb_acc_10b4_fixed_joint
- removed joint l_upper_leg_mtb_acc_10b5_fixed_joint
- removed joint l_upper_leg_mtb_acc_10b6_fixed_joint
- removed joint l_upper_leg_mtb_acc_10b7_fixed_joint
- removed joint r_foot_mtb_acc_11b12_fixed_joint
- removed joint r_foot_mtb_acc_11b13_fixed_joint
- removed joint r_forearm_mtb_acc_2b7_fixed_joint
- removed joint r_forearm_mtb_acc_2b8_fixed_joint
- removed joint r_forearm_mtb_acc_2b9_fixed_joint
- removed joint r_lower_leg_ems_acc_eb9_fixed_joint
- removed joint r_lower_leg_ems_gyro_eb9_fixed_joint
- removed joint r_lower_leg_mtb_acc_11b10_fixed_joint
- removed joint r_lower_leg_mtb_acc_11b11_fixed_joint
- removed joint r_lower_leg_mtb_acc_11b8_fixed_joint
- removed joint r_lower_leg_mtb_acc_11b9_fixed_joint
- removed joint r_upper_arm_mtb_acc_2b10_fixed_joint
- removed joint r_upper_arm_mtb_acc_2b11_fixed_joint
- removed joint r_upper_arm_mtb_acc_2b12_fixed_joint
- removed joint r_upper_arm_mtb_acc_2b13_fixed_joint
- removed joint r_upper_leg_ems_acc_eb11_fixed_joint
- removed joint r_upper_leg_ems_acc_eb8_fixed_joint
- removed joint r_upper_leg_ems_gyro_eb11_fixed_joint
- removed joint r_upper_leg_ems_gyro_eb8_fixed_joint
- removed joint r_upper_leg_mtb_acc_11b1_fixed_joint
- removed joint r_upper_leg_mtb_acc_11b2_fixed_joint
- removed joint r_upper_leg_mtb_acc_11b3_fixed_joint
- removed joint r_upper_leg_mtb_acc_11b4_fixed_joint
- removed joint r_upper_leg_mtb_acc_11b5_fixed_joint
- removed joint r_upper_leg_mtb_acc_11b6_fixed_joint
- removed joint r_upper_leg_mtb_acc_11b7_fixed_joint
- removed joint root_link_ems_acc_eb5_fixed_joint
- removed joint root_link_ems_gyro_eb5_fixed_joint
- added joint imu_frame_fixed_joint: type fixed, parent head, child imu_frame, origin xyz=0.00950000019074 0.133444 0.0093 rpy=-1.57079632679 1.57079632679 0
- joint r_wrist_prosup: axis -0.965925843882 2.22044604925e-16 0.258818979447 -> 0.965925843882 -2.22044604925e-16 -0.258818979447

File: iCub/robots/iCubGenova02/model.urdf (robot description, URDF)
Before this commit: robot ICUB_2-5_BB_SIM_MODEL, 163 links, 162 joints
Links:
- removed link chest_ems_acc_eb1
- removed link chest_ems_acc_eb2
- removed link chest_ems_acc_eb3
- removed link chest_ems_acc_eb4
- removed link chest_ems_gyro_eb1
- removed link chest_ems_gyro_eb2
- removed link chest_ems_gyro_eb3
- removed link chest_ems_gyro_eb4
- removed link chest_mtb_acc_0b10
- removed link chest_mtb_acc_0b7
- removed link chest_mtb_acc_0b8
- removed link chest_mtb_acc_0b9
- removed link l_foot_mtb_acc_10b12
- removed link l_foot_mtb_acc_10b13
- removed link l_forearm_mtb_acc_1b7
- removed link l_forearm_mtb_acc_1b8
- removed link l_forearm_mtb_acc_1b9
- removed link l_lower_leg_ems_acc_eb7
- removed link l_lower_leg_ems_gyro_eb7
- removed link l_lower_leg_mtb_acc_10b10
- removed link l_lower_leg_mtb_acc_10b11
- removed link l_lower_leg_mtb_acc_10b8
- removed link l_lower_leg_mtb_acc_10b9
- removed link l_upper_arm_mtb_acc_1b10
- removed link l_upper_arm_mtb_acc_1b11
- removed link l_upper_arm_mtb_acc_1b12
- removed link l_upper_arm_mtb_acc_1b13
- removed link l_upper_leg_ems_acc_eb10
- removed link l_upper_leg_ems_acc_eb6
- removed link l_upper_leg_ems_gyro_eb10
- removed link l_upper_leg_ems_gyro_eb6
- removed link l_upper_leg_mtb_acc_10b1
- removed link l_upper_leg_mtb_acc_10b2
- removed link l_upper_leg_mtb_acc_10b3
- removed link l_upper_leg_mtb_acc_10b4
- removed link l_upper_leg_mtb_acc_10b5
- removed link l_upper_leg_mtb_acc_10b6
- removed link l_upper_leg_mtb_acc_10b7
- removed link r_foot_mtb_acc_11b12
- removed link r_foot_mtb_acc_11b13
- removed link r_forearm_mtb_acc_2b7
- removed link r_forearm_mtb_acc_2b8
- removed link r_forearm_mtb_acc_2b9
- removed link r_lower_leg_ems_acc_eb9
- removed link r_lower_leg_ems_gyro_eb9
- removed link r_lower_leg_mtb_acc_11b10
- removed link r_lower_leg_mtb_acc_11b11
- removed link r_lower_leg_mtb_acc_11b8
- removed link r_lower_leg_mtb_acc_11b9
- removed link r_upper_arm_mtb_acc_2b10
- removed link r_upper_arm_mtb_acc_2b11
- removed link r_upper_arm_mtb_acc_2b12
- removed link r_upper_arm_mtb_acc_2b13
- removed link r_upper_leg_ems_acc_eb11
- removed link r_upper_leg_ems_acc_eb8
- removed link r_upper_leg_ems_gyro_eb11
- removed link r_upper_leg_ems_gyro_eb8
- removed link r_upper_leg_mtb_acc_11b1
- removed link r_upper_leg_mtb_acc_11b2
- removed link r_upper_leg_mtb_acc_11b3
- removed link r_upper_leg_mtb_acc_11b4
- removed link r_upper_leg_mtb_acc_11b5
- removed link r_upper_leg_mtb_acc_11b6
- removed link r_upper_leg_mtb_acc_11b7
- removed link root_link_ems_acc_eb5
- removed link root_link_ems_gyro_eb5
Joints:
- removed joint chest_ems_acc_eb1_fixed_joint
- removed joint chest_ems_acc_eb2_fixed_joint
- removed joint chest_ems_acc_eb3_fixed_joint
- removed joint chest_ems_acc_eb4_fixed_joint
- removed joint chest_ems_gyro_eb1_fixed_joint
- removed joint chest_ems_gyro_eb2_fixed_joint
- removed joint chest_ems_gyro_eb3_fixed_joint
- removed joint chest_ems_gyro_eb4_fixed_joint
- removed joint chest_mtb_acc_0b10_fixed_joint
- removed joint chest_mtb_acc_0b7_fixed_joint
- removed joint chest_mtb_acc_0b8_fixed_joint
- removed joint chest_mtb_acc_0b9_fixed_joint
- removed joint l_foot_mtb_acc_10b12_fixed_joint
- removed joint l_foot_mtb_acc_10b13_fixed_joint
- removed joint l_forearm_mtb_acc_1b7_fixed_joint
- removed joint l_forearm_mtb_acc_1b8_fixed_joint
- removed joint l_forearm_mtb_acc_1b9_fixed_joint
- removed joint l_lower_leg_ems_acc_eb7_fixed_joint
- removed joint l_lower_leg_ems_gyro_eb7_fixed_joint
- removed joint l_lower_leg_mtb_acc_10b10_fixed_joint
- removed joint l_lower_leg_mtb_acc_10b11_fixed_joint
- removed joint l_lower_leg_mtb_acc_10b8_fixed_joint
- removed joint l_lower_leg_mtb_acc_10b9_fixed_joint
- removed joint l_upper_arm_mtb_acc_1b10_fixed_joint
- removed joint l_upper_arm_mtb_acc_1b11_fixed_joint
- removed joint l_upper_arm_mtb_acc_1b12_fixed_joint
- removed joint l_upper_arm_mtb_acc_1b13_fixed_joint
- removed joint l_upper_leg_ems_acc_eb10_fixed_joint
- removed joint l_upper_leg_ems_acc_eb6_fixed_joint
- removed joint l_upper_leg_ems_gyro_eb10_fixed_joint
- removed joint l_upper_leg_ems_gyro_eb6_fixed_joint
- removed joint l_upper_leg_mtb_acc_10b1_fixed_joint
- removed joint l_upper_leg_mtb_acc_10b2_fixed_joint
- removed joint l_upper_leg_mtb_acc_10b3_fixed_joint
- removed joint l_upper_leg_mtb_acc_10b4_fixed_joint
- removed joint l_upper_leg_mtb_acc_10b5_fixed_joint
- removed joint l_upper_leg_mtb_acc_10b6_fixed_joint
- removed joint l_upper_leg_mtb_acc_10b7_fixed_joint
- removed joint r_foot_mtb_acc_11b12_fixed_joint
- removed joint r_foot_mtb_acc_11b13_fixed_joint
- removed joint r_forearm_mtb_acc_2b7_fixed_joint
- removed joint r_forearm_mtb_acc_2b8_fixed_joint
- removed joint r_forearm_mtb_acc_2b9_fixed_joint
- removed joint r_lower_leg_ems_acc_eb9_fixed_joint
- removed joint r_lower_leg_ems_gyro_eb9_fixed_joint
- removed joint r_lower_leg_mtb_acc_11b10_fixed_joint
- removed joint r_lower_leg_mtb_acc_11b11_fixed_joint
- removed joint r_lower_leg_mtb_acc_11b8_fixed_joint
- removed joint r_lower_leg_mtb_acc_11b9_fixed_joint
- removed joint r_upper_arm_mtb_acc_2b10_fixed_joint
- removed joint r_upper_arm_mtb_acc_2b11_fixed_joint
- removed joint r_upper_arm_mtb_acc_2b12_fixed_joint
- removed joint r_upper_arm_mtb_acc_2b13_fixed_joint
- removed joint r_upper_leg_ems_acc_eb11_fixed_joint
- removed joint r_upper_leg_ems_acc_eb8_fixed_joint
- removed joint r_upper_leg_ems_gyro_eb11_fixed_joint
- removed joint r_upper_leg_ems_gyro_eb8_fixed_joint
- removed joint r_upper_leg_mtb_acc_11b1_fixed_joint
- removed joint r_upper_leg_mtb_acc_11b2_fixed_joint
- removed joint r_upper_leg_mtb_acc_11b3_fixed_joint
- removed joint r_upper_leg_mtb_acc_11b4_fixed_joint
- removed joint r_upper_leg_mtb_acc_11b5_fixed_joint
- removed joint r_upper_leg_mtb_acc_11b6_fixed_joint
- removed joint r_upper_leg_mtb_acc_11b7_fixed_joint
- removed joint root_link_ems_acc_eb5_fixed_joint
- removed joint root_link_ems_gyro_eb5_fixed_joint
