Commit message: Updated models

File: iCub/robots/iCubGenova04/model.urdf (robot description, URDF)
Before this commit: robot ICUB_2-5_BB_SIM_MODEL, 163 links, 162 joints
Links:
- removed link chest_ems_acc_eb1
- removed link chest_ems_acc_eb2
- removed link chest_ems_acc_eb3
- removed link chest_ems_acc_eb4
- removed link chest_ems_gyro_eb1
- removed link chest_ems_gyro_eb2
- removed link chest_ems_gyro_eb3
- removed link chest_ems_gyro_eb4
- removed link chest_mtb_acc_0b10
- removed link chest_mtb_acc_0b7
- removed link chest_mtb_acc_0b8
- removed link chest_mtb_acc_0b9
- removed link l_foot_mtb_acc_10b12
- removed link l_foot_mtb_acc_10b13
- removed link l_forearm_mtb_acc_1b7
- removed link l_forearm_mtb_acc_1b8
- removed link l_forearm_mtb_acc_1b9
- removed link l_lower_leg_ems_acc_eb7
- removed link l_lower_leg_ems_gyro_eb7
- removed link l_lower_leg_mtb_acc_10b10
- removed link l_lower_leg_mtb_acc_10b11
- removed link l_lower_leg_mtb_acc_10b8
- removed link l_lower_leg_mtb_acc_10b9
- removed link l_upper_arm_mtb_acc_1b10
- removed link l_upper_arm_mtb_acc_1b11
- removed link l_upper_arm_mtb_acc_1b12
- removed link l_upper_arm_mtb_acc_1b13
- removed link l_upper_leg_ems_acc_eb10
- removed link l_upper_leg_ems_acc_eb6
- removed link l_upper_leg_ems_gyro_eb10
- removed link l_upper_leg_ems_gyro_eb6
- removed link l_upper_leg_mtb_acc_10b1
- removed link l_upper_leg_mtb_acc_10b2
- removed link l_upper_leg_mtb_acc_10b3
- removed link l_upper_leg_mtb_acc_10b4
- removed link l_upper_leg_mtb_acc_10b5
- removed link l_upper_leg_mtb_acc_10b6
- removed link l_upper_leg_mtb_acc_10b7
- removed link r_foot_mtb_acc_11b12
- removed link r_foot_mtb_acc_11b13
- removed link r_forearm_mtb_acc_2b7
- removed link r_forearm_mtb_acc_2b8
- removed link r_forearm_mtb_acc_2b9
- removed link r_lower_leg_ems_acc_eb9
- removed link r_lower_leg_ems_gyro_eb9
- removed link r_lower_leg_mtb_acc_11b10
- removed link r_lower_leg_mtb_acc_11b11
- removed link r_lower_leg_mtb_acc_11b8
- removed link r_lower_leg_mtb_acc_11b9
- removed link r_upper_arm_mtb_acc_2b10
- removed link r_upper_arm_mtb_acc_2b11
- removed link r_upper_arm_mtb_acc_2b12
- removed link r_upper_arm_mtb_acc_2b13
- removed link r_upper_leg_ems_acc_eb11
- removed link r_upper_leg_ems_acc_eb8
- removed link r_upper_leg_ems_gyro_eb11
- removed link r_upper_leg_ems_gyro_eb8
- removed link r_upper_leg_mtb_acc_11b1
- removed link r_upper_leg_mtb_acc_11b2
- removed link r_upper_leg_mtb_acc_11b3
- removed link r_upper_leg_mtb_acc_11b4
- removed link r_upper_leg_mtb_acc_11b5
- removed link r_upper_leg_mtb_acc_11b6
- removed link r_upper_leg_mtb_acc_11b7
- removed link root_link_ems_acc_eb5
- removed link root_link_ems_gyro_eb5
Joints:
- removed joint chest_ems_acc_eb1_fixed_joint
- removed joint chest_ems_acc_eb2_fixed_joint
- removed joint chest_ems_acc_eb3_fixed_joint
- removed joint chest_ems_acc_eb4_fixed_joint
- removed joint chest_ems_gyro_eb1_fixed_joint
- removed joint chest_ems_gyro_eb2_fixed_joint
- removed joint chest_ems_gyro_eb3_fixed_joint
- removed joint chest_ems_gyro_eb4_fixed_joint
- removed joint chest_mtb_acc_0b10_fixed_joint
- removed joint chest_mtb_acc_0b7_fixed_joint
- removed joint chest_mtb_acc_0b8_fixed_joint
- removed joint chest_mtb_acc_0b9_fixed_joint
- removed joint l_foot_mtb_acc_10b12_fixed_joint
- removed joint l_foot_mtb_acc_10b13_fixed_joint
- removed joint l_forearm_mtb_acc_1b7_fixed_joint
- removed joint l_forearm_mtb_acc_1b8_fixed_joint
- removed joint l_forearm_mtb_acc_1b9_fixed_joint
- removed joint l_lower_leg_ems_acc_eb7_fixed_joint
- removed joint l_lower_leg_ems_gyro_eb7_fixed_joint
- removed joint l_lower_leg_mtb_acc_10b10_fixed_joint
- removed joint l_lower_leg_mtb_acc_10b11_fixed_joint
- removed joint l_lower_leg_mtb_acc_10b8_fixed_joint
- removed joint l_lower_leg_mtb_acc_10b9_fixed_joint
- removed joint l_upper_arm_mtb_acc_1b10_fixed_joint
- removed joint l_upper_arm_mtb_acc_1b11_fixed_joint
- removed joint l_upper_arm_mtb_acc_1b12_fixed_joint
- removed joint l_upper_arm_mtb_acc_1b13_fixed_joint
- removed joint l_upper_leg_ems_acc_eb10_fixed_joint
- removed joint l_upper_leg_ems_acc_eb6_fixed_joint
- removed joint l_upper_leg_ems_gyro_eb10_fixed_joint
- removed joint l_upper_leg_ems_gyro_eb6_fixed_joint
- removed joint l_upper_leg_mtb_acc_10b1_fixed_joint
- removed joint l_upper_leg_mtb_acc_10b2_fixed_joint
- removed joint l_upper_leg_mtb_acc_10b3_fixed_joint
- removed joint l_upper_leg_mtb_acc_10b4_fixed_joint
- removed joint l_upper_leg_mtb_acc_10b5_fixed_joint
- removed joint l_upper_leg_mtb_acc_10b6_fixed_joint
- removed joint l_upper_leg_mtb_acc_10b7_fixed_joint
- removed joint r_foot_mtb_acc_11b12_fixed_joint
- removed joint r_foot_mtb_acc_11b13_fixed_joint
- removed joint r_forearm_mtb_acc_2b7_fixed_joint
- removed joint r_forearm_mtb_acc_2b8_fixed_joint
- removed joint r_forearm_mtb_acc_2b9_fixed_joint
- removed joint r_lower_leg_ems_acc_eb9_fixed_joint
- removed joint r_lower_leg_ems_gyro_eb9_fixed_joint
- removed joint r_lower_leg_mtb_acc_11b10_fixed_joint
- removed joint r_lower_leg_mtb_acc_11b11_fixed_joint
- removed joint r_lower_leg_mtb_acc_11b8_fixed_joint
- removed joint r_lower_leg_mtb_acc_11b9_fixed_joint
- removed joint r_upper_arm_mtb_acc_2b10_fixed_joint
- removed joint r_upper_arm_mtb_acc_2b11_fixed_joint
- removed joint r_upper_arm_mtb_acc_2b12_fixed_joint
- removed joint r_upper_arm_mtb_acc_2b13_fixed_joint
- removed joint r_upper_leg_ems_acc_eb11_fixed_joint
- removed joint r_upper_leg_ems_acc_eb8_fixed_joint
- removed joint r_upper_leg_ems_gyro_eb11_fixed_joint
- removed joint r_upper_leg_ems_gyro_eb8_fixed_joint
- removed joint r_upper_leg_mtb_acc_11b1_fixed_joint
- removed joint r_upper_leg_mtb_acc_11b2_fixed_joint
- removed joint r_upper_leg_mtb_acc_11b3_fixed_joint
- removed joint r_upper_leg_mtb_acc_11b4_fixed_joint
- removed joint r_upper_leg_mtb_acc_11b5_fixed_joint
- removed joint r_upper_leg_mtb_acc_11b6_fixed_joint
- removed joint r_upper_leg_mtb_acc_11b7_fixed_joint
- removed joint root_link_ems_acc_eb5_fixed_joint
- removed joint root_link_ems_gyro_eb5_fixed_joint
