Commit message: Fixed hip and ankle joints limits.

File: iCub/robots/iCubGenova04/model.urdf (robot description, URDF)
Before this commit: robot iCub, 97 links, 96 joints
Joints:
- joint l_ankle_pitch: limit lower=-0.349065850399 upper=0.523598775598 effort=50000 velocity=50000 -> lower=-0.523598775598 upper=0.523598775598 effort=50000 velocity=50000
- joint l_hip_roll: limit lower=0.0 upper=1.57079632679 effort=50000 velocity=50000 -> lower=-0.261799 upper=1.482777778 effort=50000 velocity=50000
- joint r_ankle_pitch: limit lower=-0.349065850399 upper=0.523598775598 effort=50000 velocity=50000 -> lower=-0.523598775598 upper=0.523598775598 effort=50000 velocity=50000
- joint r_hip_roll: limit lower=0.0 upper=1.57079632679 effort=50000 velocity=50000 -> lower=-0.261799 upper=1.482777778 effort=50000 velocity=50000
